File: TPS63031.kicad_pcb (KiCad board)
At the start: 2 copper layers, 22 x 15 mm, 10 parts, among them J1 Conn_01x03, J2 Conn_01x03, U1 TPS63031

Commit message: Inductor type specification
Parts:
- L1: value L -> 74438334015
Changed lines of the file:
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@@
       (effects (font (size 1 1) (thickness 0.15)))
     )
-    (fp_text value L (at 0 3.2) (layer F.Fab)
+    (fp_text value 74438334015 (at 0 3.2) (layer F.Fab)
       (effects (font (size 1 1) (thickness 0.15)))
     )
